Commit message: Save grasp collection, evaluation, and workspace artifacts

File: assets/stack_box/box.urdf (robot description, URDF)
Before this commit: robot stack_box, 5 links, 4 joints
Links:
- added link bottom; collision box size=0.25 0.30 0.01; visual box size=0.25 0.30 0.01
- link box_root: geometry 
- link wall_x0: geometry collision box size=0.01 0.30 0.30; visual box size=0.01 0.30 0.30
- link wall_x1: geometry collision box size=0.01 0.30 0.30; visual box size=0.01 0.30 0.30
- link wall_y0: geometry collision box size=0.25 0.01 0.30; visual box size=0.25 0.01 0.30
- link wall_y1: geometry collision box size=0.25 0.01 0.30; visual box size=0.25 0.01 0.30
Joints:
- added joint bottom_joint: type fixed, parent box_root, child bottom, origin xyz=0.1254 0 0.1665
- joint wall_x0_joint: origin xyz=-0.145 0 0.055 -> xyz=0.0059 0 0.091
- joint wall_x1_joint: origin xyz=0.145 0 0.055 -> xyz=0.245 0 0.0936
- joint wall_y0_joint: origin xyz=0 -0.105 0.055 -> xyz=0.1255 -0.1434 0.0914
- joint wall_y1_joint: origin xyz=0 0.105 0.055 -> xyz=0.1207 0.1462 0.094
